File: PressureSensors/LPS22HB/LPS22HB_pcb.brd (EAGLE design)
At the start: 3.9 x 5.4 mm, 7 parts

Commit message: pressure sensor changes
Parts:
- removed C1: 100nF, resistor:C0201
- added C2: 100nF, resistor:C0402
Connections:
- net +3V3: now also C2.1; no longer C1.1
- net GND: now also C2.2; no longer C1.2
Routing:
- net GND: track 9.22 -> 9.92 mm
- net +3V3: track 5.63 -> 5.03 mm
Other:
- board outline removed
Changed lines of the file:
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@@
 <setting verticaltext="up"/>
 </settings>
-<grid distance="0.05" unitdist="mm" unit="mm" style="lines" multiple="1" display="yes" altdistance="5" altunitdist="mil" altunit="mil"/>
+<grid distance="0.15" unitdist="mil" unit="mil" style="lines" multiple="1" display="yes" altdistance="5" altunitdist="mil" altunit="mil"/>
 <layers>
 <layer number="1" name="Top" color="4" fill="1" visible="yes" active="yes"/>
@@
 <board>
 <plain>
-<wire x1="0" y1="0" x2="3.85" y2="0" width="0" layer="20"/>
-<wire x1="3.85" y1="0" x2="3.85" y2="5.4" width="0" layer="20"/>
-<wire x1="3.85" y1="5.4" x2="0" y2="5.4" width="0" layer="20"/>
-<wire x1="0" y1="5.4" x2="0" y2="0" width="0" layer="20"/>
 <text x="2.2" y="1.95" size="0.254" layer="22" rot="MR90">100nF</text>
 <wire x1="0.1" y1="5.3" x2="0.1" y2="0.1" width="0.15" layer="21"/>
@@
 <element name="U$7" library="wirepad_08-045" package="WIREPAD_0,8/0,45" value="WIREPAD_0,8/0,45" x="1.9" y="4.7"/>
 <element name="U$8" library="wirepad_08-045" package="WIREPAD_0,8/0,45" value="WIREPAD_0,8/0,45" x="0.785" y="4.2"/>
-<element name="C1" library="resistor" library_urn="urn:adsk.eagle:library:348" package="C0201" value="100nF" x="1.9" y="2.5" smashed="yes" rot="MR270"/>
 <element name="U$1" library="LPS22HB" package="LPS22HB_HLGA" value="LPS22HB_HLGA" x="1.9" y="2.5" rot="R180"/>
+<element name="C2" library="resistor" library_urn="urn:adsk.eagle:library:348" package="C0402" value="100nF" x="1.477090625" y="2.49285" smashed="yes" rot="MR270"/>
 </elements>
 <signals>
 <signal name="+3V3">
 <contactref element="U$8" pad="P$1"/>
-<contactref element="C1" pad="1"/>
 <contactref element="U$1" pad="P$1"/>
 <contactref element="U$1" pad="P$10"/>
@@
 <wire x1="1.4" y1="3.6" x2="1.4" y2="3.2625" width="0.1524" layer="1"/>
 <wire x1="0.785" y1="4.2" x2="1.4" y2="3.6" width="0.1524" layer="1"/>
-<wire x1="0.80060625" y1="3.74939375" x2="1.65" y2="2.9" width="0.1524" layer="16"/>
-<wire x1="1.65" y1="2.9" x2="1.9" y2="2.75" width="0.1524" layer="16"/>
 <wire x1="2.6625" y1="2.25" x2="1.7125" y2="2.6" width="0.1524" layer="1"/>
 <wire x1="1.7125" y1="2.6" x2="1.1375" y2="2.75" width="0.1524" layer="1"/>
-<wire x1="0.785" y1="4.2" x2="0.80060625" y2="3.74939375" width="0.1524" layer="16"/>
+<contactref element="C2" pad="1"/>
+<wire x1="0.785" y1="4.2" x2="0.785" y2="3.834940625" width="0.1524" layer="16"/>
+<wire x1="0.785" y1="3.834940625" x2="1.477090625" y2="3.14285" width="0.1524" layer="16"/>
 </signal>
 <signal name="GND">
 <contactref element="U$7" pad="P$1"/>
-<contactref element="C1" pad="2"/>
 <contactref element="U$1" pad="P$9"/>
 <contactref element="U$1" pad="P$8"/>
@@
 <wire x1="1.9" y1="3.2625" x2="2.4" y2="3.2625" width="0.1524" layer="1"/>
 <wire x1="1.9" y1="4.7" x2="1.9" y2="3.2625" width="0.1524" layer="1"/>
-<wire x1="1.9" y1="4.7" x2="1.9" y2="3.55" width="0.1524" layer="16"/>
-<wire x1="1.9" y1="3.55" x2="2.4" y2="3.05" width="0.1524" layer="16"/>
-<wire x1="2.4" y1="3.05" x2="2.4" y2="2.25" width="0.1524" layer="16"/>
-<wire x1="2.4" y1="2.25" x2="1.9" y2="2.25" width="0.1524" layer="16"/>
-<wire x1="1.9" y1="2.25" x2="1.9" y2="0.7" width="0.1524" layer="16"/>
 <via x="1.9" y="0.7" extent="1-16" drill="0.35"/>
 <wire x1="1.4" y1="1.3375" x2="1.4" y2="1.7375" width="0.1524" layer="1"/>
 <wire x1="1.4" y1="1.3375" x2="1.9" y2="0.7" width="0.1524" layer="1"/>
-<wire x1="1.4" y1="1.7375" x2="1.65" y2="2.1" width="0.1524" layer="1"/>
-<wire x1="1.65" y1="2.1" x2="2.1" y2="2.1" width="0.1524" layer="1"/>
-<wire x1="2.1" y1="2.1" x2="2.4" y2="1.7375" width="0.1524" layer="1"/>
+<contactref element="C2" pad="2"/>
+<wire x1="1.4" y1="1.7375" x2="1.4" y2="1.85" width="0.1524" layer="1"/>
+<wire x1="1.4" y1="1.85" x2="1.75" y2="2.2" width="0.1524" layer="1"/>
+<wire x1="2.1196875" y1="2.1036" x2="2.2536" y2="1.9696875" width="0.1524" layer="1"/>
+<wire x1="2.2536" y1="1.9696875" x2="2.2536" y2="1.8839" width="0.1524" layer="1"/>
+<wire x1="2.2536" y1="1.8839" x2="2.4" y2="1.7375" width="0.1524" layer="1"/>
+<wire x1="1.8580375" y1="2.2" x2="2.1196875" y2="2.1036" width="0.1524" layer="1"/>
+<wire x1="1.75" y1="2.2" x2="1.8580375" y2="2.2" width="0.1524" layer="1"/>
+<wire x1="1.9" y1="4.25" x2="1.9" y2="4.7" width="0.1524" layer="16"/>
+<wire x1="1.9" y1="0.7" x2="1.9" y2="1.419940625" width="0.1524" layer="16"/>
+<wire x1="1.477090625" y1="1.84285" x2="1.9" y2="1.419940625" width="0.1524" layer="16"/>
+<wire x1="1.9" y1="4.7" x2="1.9" y2="3.95596875" width="0.1524" layer="16"/>
+<wire x1="1.9" y1="3.95596875" x2="2.49555" y2="3.36041875" width="0.1524" layer="16"/>
+<wire x1="2.49555" y1="3.36041875" x2="2.49555" y2="2.861309375" width="0.1524" layer="16"/>
+<wire x1="2.49555" y1="2.861309375" x2="1.477090625" y2="1.84285" width="0.1524" layer="16"/>
 </signal>
 <signal name="N$4">
@@
 </signal>
 </signals>
+<errors>
+</errors>
 </board>
 </drawing>
