File: PressureSensors/Amphenol_NPA201/amphenol_npa201.brd (EAGLE design)
At the start: 6.1 x 3 mm, 5 parts

Commit message: pressure sensor changes
Parts:
- moved U$1 6.41 mm to (7.95, 5.49)
- moved U$4 6.40 mm to (10.2, 6.11)
- moved U$5 6.40 mm to (10.2, 4.86)
- moved U$2 6.40 mm to (5.75, 6.11)
- moved U$3 6.40 mm to (5.75, 4.86)
Other:
- board outline removed
Changed lines of the file:
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@@
 <setting verticaltext="up"/>
 </settings>
-<grid distance="0.01" unitdist="mm" unit="mm" style="lines" multiple="1" display="yes" altdistance="5" altunitdist="mil" altunit="mil"/>
+<grid distance="1" unitdist="mil" unit="mil" style="lines" multiple="1" display="yes" altdistance="5" altunitdist="mil" altunit="mil"/>
 <layers>
 <layer number="1" name="Top" color="4" fill="1" visible="yes" active="yes"/>
@@
 <layer number="27" name="tValues" color="7" fill="1" visible="yes" active="yes"/>
 <layer number="28" name="bValues" color="7" fill="1" visible="yes" active="yes"/>
-<layer number="29" name="tStop" color="7" fill="3" visible="no" active="yes"/>
-<layer number="30" name="bStop" color="7" fill="6" visible="no" active="yes"/>
-<layer number="31" name="tCream" color="7" fill="4" visible="no" active="yes"/>
-<layer number="32" name="bCream" color="7" fill="5" visible="no" active="yes"/>
-<layer number="33" name="tFinish" color="6" fill="3" visible="no" active="yes"/>
-<layer number="34" name="bFinish" color="6" fill="6" visible="no" active="yes"/>
-<layer number="35" name="tGlue" color="7" fill="4" visible="no" active="yes"/>
-<layer number="36" name="bGlue" color="7" fill="5" visible="no" active="yes"/>
-<layer number="37" name="tTest" color="7" fill="1" visible="no" active="yes"/>
-<layer number="38" name="bTest" color="7" fill="1" visible="no" active="yes"/>
+<layer number="29" name="tStop" color="7" fill="3" visible="yes" active="yes"/>
+<layer number="30" name="bStop" color="7" fill="6" visible="yes" active="yes"/>
+<layer number="31" name="tCream" color="7" fill="4" visible="yes" active="yes"/>
+<layer number="32" name="bCream" color="7" fill="5" visible="yes" active="yes"/>
+<layer number="33" name="tFinish" color="6" fill="3" visible="yes" active="yes"/>
+<layer number="34" name="bFinish" color="6" fill="6" visible="yes" active="yes"/>
+<layer number="35" name="tGlue" color="7" fill="4" visible="yes" active="yes"/>
+<layer number="36" name="bGlue" color="7" fill="5" visible="yes" active="yes"/>
+<layer number="37" name="tTest" color="7" fill="1" visible="yes" active="yes"/>
+<layer number="38" name="bTest" color="7" fill="1" visible="yes" active="yes"/>
 <layer number="39" name="tKeepout" color="4" fill="11" visible="yes" active="yes"/>
 <layer number="40" name="bKeepout" color="1" fill="11" visible="yes" active="yes"/>
@@
 <layer number="42" name="bRestrict" color="1" fill="10" visible="yes" active="yes"/>
 <layer number="43" name="vRestrict" color="2" fill="10" visible="yes" active="yes"/>
-<layer number="44" name="Drills" color="7" fill="1" visible="no" active="yes"/>
+<layer number="44" name="Drills" color="7" fill="1" visible="yes" active="yes"/>
 <layer number="45" name="Holes" color="7" fill="1" visible="yes" active="yes"/>
-<layer number="46" name="Milling" color="3" fill="1" visible="no" active="yes"/>
-<layer number="47" name="Measures" color="7" fill="1" visible="no" active="yes"/>
+<layer number="46" name="Milling" color="3" fill="1" visible="yes" active="yes"/>
+<layer number="47" name="Measures" color="7" fill="1" visible="yes" active="yes"/>
 <layer number="48" name="Document" color="7" fill="1" visible="yes" active="yes"/>
 <layer number="49" name="Reference" color="7" fill="1" visible="yes" active="yes"/>
@@
 <board>
 <plain>
-<wire x1="0" y1="0" x2="6.1" y2="0" width="0" layer="20"/>
-<wire x1="6.1" y1="0" x2="6.1" y2="3.05" width="0" layer="20"/>
-<wire x1="6.1" y1="3.05" x2="0" y2="3.05" width="0" layer="20"/>
-<wire x1="0" y1="3.05" x2="0" y2="0" width="0" layer="20"/>
-<wire x1="0.15" y1="2.85" x2="5.85" y2="2.85" width="0.1524" layer="21"/>
-<wire x1="5.85" y1="2.85" x2="5.85" y2="0.15" width="0.1524" layer="21"/>
-<wire x1="5.85" y1="0.15" x2="0.15" y2="0.15" width="0.1524" layer="21"/>
-<wire x1="0.15" y1="0.15" x2="0.15" y2="2.85" width="0.1524" layer="21"/>
+<wire x1="5.15" y1="6.85" x2="10.85" y2="6.85" width="0.1524" layer="21"/>
+<wire x1="10.85" y1="6.85" x2="10.85" y2="4.15" width="0.1524" layer="21"/>
+<wire x1="10.85" y1="4.15" x2="5.15" y2="4.15" width="0.1524" layer="21"/>
+<wire x1="5.15" y1="4.15" x2="5.15" y2="6.85" width="0.1524" layer="21"/>
+<circle x="9.54" y="4.42" radius="0.080621875" width="0.1524" layer="21"/>
 </plain>
 <attributes>
@@
 </autorouter>
 <elements>
-<element name="U$1" library="Amphenol_NPA201" package="AMPHENOL_NPA201" value="AMPHENOL_NPA201" x="2.96" y="1.47"/>
-<element name="U$2" library="wirepad_08-045" package="WIREPAD_0,8/0,45" value="WIREPAD_0,8/0,45" x="0.75" y="2.11"/>
-<element name="U$3" library="wirepad_08-045" package="WIREPAD_0,8/0,45" value="WIREPAD_0,8/0,45" x="0.75" y="0.86"/>
-<element name="U$4" library="wirepad_08-045" package="WIREPAD_0,8/0,45" value="WIREPAD_0,8/0,45" x="5.22" y="2.11"/>
-<element name="U$5" library="wirepad_08-045" package="WIREPAD_0,8/0,45" value="WIREPAD_0,8/0,45" x="5.22" y="0.86"/>
+<element name="U$2" library="wirepad_08-045" package="WIREPAD_0,8/0,45" value="WIREPAD_0,8/0,45" x="5.75" y="6.11"/>
+<element name="U$3" library="wirepad_08-045" package="WIREPAD_0,8/0,45" value="WIREPAD_0,8/0,45" x="5.75" y="4.86"/>
+<element name="U$4" library="wirepad_08-045" package="WIREPAD_0,8/0,45" value="WIREPAD_0,8/0,45" x="10.22" y="6.11"/>
+<element name="U$5" library="wirepad_08-045" package="WIREPAD_0,8/0,45" value="WIREPAD_0,8/0,45" x="10.22" y="4.86"/>
+<element name="U$1" library="Amphenol_NPA201" package="AMPHENOL_NPA201" value="AMPHENOL_NPA201" x="7.95" y="5.49"/>
 </elements>
 <signals>
 <signal name="GND">
+<contactref element="U$5" pad="P$1"/>
 <contactref element="U$1" pad="P$1"/>
-<contactref element="U$5" pad="P$1"/>
 <contactref element="U$1" pad="P$7"/>
-<wire x1="3.285" y1="2.195" x2="3.485" y2="1.595" width="0.1524" layer="1"/>
-<wire x1="3.485" y1="1.595" x2="3.935" y2="0.745" width="0.1524" layer="1"/>
-<wire x1="3.935" y1="0.745" x2="4.825" y2="0.745" width="0.1524" layer="1"/>
-<wire x1="4.825" y1="0.745" x2="5.22" y2="0.86" width="0.1524" layer="1"/>
+<wire x1="8.275" y1="6.215" x2="8.275" y2="5.415" width="0.1524" layer="1"/>
+<wire x1="8.275" y1="5.415" x2="8.925" y2="4.765" width="0.1524" layer="1"/>
+<wire x1="8.925" y1="4.765" x2="10.125" y2="4.765" width="0.1524" layer="1"/>
+<wire x1="10.125" y1="4.765" x2="10.22" y2="4.86" width="0.1524" layer="1"/>
 </signal>
 <signal name="N$1">
 <contactref element="U$2" pad="P$1"/>
 <contactref element="U$1" pad="P$3"/>
-<wire x1="2.635" y1="0.745" x2="2.635" y2="1.215" width="0.1524" layer="1"/>
-<wire x1="2.635" y1="1.215" x2="2.55" y2="1.3" width="0.1524" layer="1"/>
-<wire x1="2.55" y1="1.3" x2="2" y2="1.5" width="0.1524" layer="1"/>
-<wire x1="2" y1="1.5" x2="1.9" y2="1.57" width="0.1524" layer="1"/>
-<wire x1="1.9" y1="1.57" x2="0.75" y2="2.11" width="0.1524" layer="1"/>
+<wire x1="5.75" y1="6.11" x2="6.28" y2="6.11" width="0.1524" layer="1"/>
+<wire x1="6.28" y1="6.11" x2="7.625" y2="4.765" width="0.1524" layer="1"/>
 </signal>
 <signal name="N$2">
 <contactref element="U$3" pad="P$1"/>
 <contactref element="U$1" pad="P$4"/>
-<wire x1="1.985" y1="0.745" x2="1.145" y2="0.745" width="0.1524" layer="1"/>
-<wire x1="1.145" y1="0.745" x2="0.75" y2="0.86" width="0.1524" layer="1"/>
+<wire x1="5.75" y1="4.86" x2="6.88" y2="4.86" width="0.1524" layer="1"/>
+<wire x1="6.88" y1="4.86" x2="6.975" y2="4.765" width="0.1524" layer="1"/>
 </signal>
 <signal name="+3V3">
+<contactref element="U$4" pad="P$1"/>
 <contactref element="U$1" pad="P$6"/>
-<contactref element="U$4" pad="P$1"/>
 <contactref element="U$1" pad="P$8"/>
-<wire x1="3.935" y1="2.195" x2="4.945" y2="2.145" width="0.1524" layer="1"/>
-<wire x1="4.945" y1="2.145" x2="5.22" y2="2.11" width="0.1524" layer="1"/>
-<wire x1="2.635" y1="2.285" x2="2.635" y2="2.195" width="0.1524" layer="1"/>
-<wire x1="2.635" y1="2.285" x2="2.97" y2="2.63" width="0.1524" layer="1"/>
-<wire x1="2.97" y1="2.63" x2="3.55" y2="2.63" width="0.1524" layer="1"/>
-<wire x1="3.55" y1="2.63" x2="3.935" y2="2.195" width="0.1524" layer="1"/>
+<wire x1="8.925" y1="6.215" x2="10.115" y2="6.215" width="0.1524" layer="1"/>
+<wire x1="10.115" y1="6.215" x2="10.22" y2="6.11" width="0.1524" layer="1"/>
+<wire x1="7.625" y1="6.215" x2="7.625" y2="6.2882875" width="0.1524" layer="1"/>
+<wire x1="7.625" y1="6.2882875" x2="7.8279125" y2="6.669" width="0.1524" layer="1"/>
+<wire x1="8.723678125" y1="6.669" x2="7.8279125" y2="6.669" width="0.1524" layer="1"/>
+<wire x1="8.925" y1="6.215" x2="8.925" y2="6.442278125" width="0.1524" layer="1"/>
+<wire x1="8.925" y1="6.442278125" x2="8.723678125" y2="6.669" width="0.1524" layer="1"/>
 </signal>
 </signals>

Commit message: few changes
Parts:
- moved U$5 6.60 mm to (4.97, 0.86)
- moved U$4 6.45 mm to (4.97, 2.36)
- moved U$1 6.41 mm to (2.85, 1.60)
- moved U$3 6.40 mm to (0.75, 0.86)
- moved U$2 6.25 mm to (0.75, 2.36)
Changed lines of the file:
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@@
 <setting verticaltext="up"/>
 </settings>
-<grid distance="1" unitdist="mil" unit="mil" style="lines" multiple="1" display="yes" altdistance="5" altunitdist="mil" altunit="mil"/>
+<grid distance="0.05" unitdist="mm" unit="mm" style="lines" multiple="1" display="yes" altdistance="5" altunitdist="mil" altunit="mil"/>
 <layers>
 <layer number="1" name="Top" color="4" fill="1" visible="yes" active="yes"/>
@@
 <board>
 <plain>
-<wire x1="5.15" y1="6.85" x2="10.85" y2="6.85" width="0.1524" layer="21"/>
-<wire x1="10.85" y1="6.85" x2="10.85" y2="4.15" width="0.1524" layer="21"/>
-<wire x1="10.85" y1="4.15" x2="5.15" y2="4.15" width="0.1524" layer="21"/>
-<wire x1="5.15" y1="4.15" x2="5.15" y2="6.85" width="0.1524" layer="21"/>
-<circle x="9.54" y="4.42" radius="0.080621875" width="0.1524" layer="21"/>
+<wire x1="0.023" y1="3.231" x2="5.723" y2="3.231" width="0.1524" layer="21"/>
+<wire x1="5.723" y1="3.231" x2="5.723" y2="0.023" width="0.1524" layer="21"/>
+<wire x1="5.723" y1="0.023" x2="0.023" y2="0.023" width="0.1524" layer="21"/>
+<wire x1="0.023" y1="0.023" x2="0.023" y2="3.231" width="0.1524" layer="21"/>
+<circle x="4.363" y="0.32" radius="0.080621875" width="0.1524" layer="21"/>
 </plain>
 <attributes>
@@
 </autorouter>
 <elements>
-<element name="U$2" library="wirepad_08-045" package="WIREPAD_0,8/0,45" value="WIREPAD_0,8/0,45" x="5.75" y="6.11"/>
-<element name="U$3" library="wirepad_08-045" package="WIREPAD_0,8/0,45" value="WIREPAD_0,8/0,45" x="5.75" y="4.86"/>
-<element name="U$4" library="wirepad_08-045" package="WIREPAD_0,8/0,45" value="WIREPAD_0,8/0,45" x="10.22" y="6.11"/>
-<element name="U$5" library="wirepad_08-045" package="WIREPAD_0,8/0,45" value="WIREPAD_0,8/0,45" x="10.22" y="4.86"/>
-<element name="U$1" library="Amphenol_NPA201" package="AMPHENOL_NPA201" value="AMPHENOL_NPA201" x="7.95" y="5.49"/>
+<element name="U$2" library="wirepad_08-045" package="WIREPAD_0,8/0,45" value="WIREPAD_0,8/0,45" x="0.75" y="2.364"/>
+<element name="U$3" library="wirepad_08-045" package="WIREPAD_0,8/0,45" value="WIREPAD_0,8/0,45" x="0.75" y="0.86"/>
+<element name="U$4" library="wirepad_08-045" package="WIREPAD_0,8/0,45" value="WIREPAD_0,8/0,45" x="4.966" y="2.364"/>
+<element name="U$5" library="wirepad_08-045" package="WIREPAD_0,8/0,45" value="WIREPAD_0,8/0,45" x="4.966" y="0.86"/>
+<element name="U$1" library="Amphenol_NPA201" package="AMPHENOL_NPA201" value="AMPHENOL_NPA201" x="2.85" y="1.6"/>
 </elements>
 <signals>
@@
 <contactref element="U$1" pad="P$1"/>
 <contactref element="U$1" pad="P$7"/>
-<wire x1="8.275" y1="6.215" x2="8.275" y2="5.415" width="0.1524" layer="1"/>
-<wire x1="8.275" y1="5.415" x2="8.925" y2="4.765" width="0.1524" layer="1"/>
-<wire x1="8.925" y1="4.765" x2="10.125" y2="4.765" width="0.1524" layer="1"/>
-<wire x1="10.125" y1="4.765" x2="10.22" y2="4.86" width="0.1524" layer="1"/>
+<wire x1="3.175" y1="2.325" x2="3.175" y2="1.825" width="0.1524" layer="1"/>
+<wire x1="3.175" y1="1.825" x2="3.4" y2="1.6" width="0.1524" layer="1"/>
+<wire x1="3.4" y1="1.6" x2="3.75" y2="1.6" width="0.1524" layer="1"/>
+<wire x1="3.75" y1="1.6" x2="3.8" y2="1.55" width="0.1524" layer="1"/>
+<wire x1="3.8" y1="1.55" x2="3.8" y2="0.9" width="0.1524" layer="1"/>
+<wire x1="3.8" y1="0.9" x2="3.825" y2="0.875" width="0.1524" layer="1"/>
+<wire x1="3.825" y1="0.875" x2="4.951" y2="0.875" width="0.1524" layer="1"/>
+<wire x1="4.951" y1="0.875" x2="4.966" y2="0.86" width="0.1524" layer="1"/>
 </signal>
 <signal name="N$1">
 <contactref element="U$2" pad="P$1"/>
 <contactref element="U$1" pad="P$3"/>
-<wire x1="5.75" y1="6.11" x2="6.28" y2="6.11" width="0.1524" layer="1"/>
-<wire x1="6.28" y1="6.11" x2="7.625" y2="4.765" width="0.1524" layer="1"/>
+<wire x1="0.75" y1="2.364" x2="0.786" y2="2.364" width="0.1524" layer="1"/>
+<wire x1="0.786" y1="2.364" x2="1.55" y2="1.6" width="0.1524" layer="1"/>
+<wire x1="1.55" y1="1.6" x2="2.55" y2="1.6" width="0.1524" layer="1"/>
+<wire x1="2.55" y1="1.6" x2="2.55" y2="0.9" width="0.1524" layer="1"/>
+<wire x1="2.55" y1="0.9" x2="2.525" y2="0.875" width="0.1524" layer="1"/>
 </signal>
 <signal name="N$2">
 <contactref element="U$3" pad="P$1"/>
 <contactref element="U$1" pad="P$4"/>
-<wire x1="5.75" y1="4.86" x2="6.88" y2="4.86" width="0.1524" layer="1"/>
-<wire x1="6.88" y1="4.86" x2="6.975" y2="4.765" width="0.1524" layer="1"/>
+<wire x1="0.75" y1="0.86" x2="1.86" y2="0.86" width="0.1524" layer="1"/>
+<wire x1="1.86" y1="0.86" x2="1.875" y2="0.875" width="0.1524" layer="1"/>
 </signal>
 <signal name="+3V3">
@@
 <contactref element="U$1" pad="P$6"/>
 <contactref element="U$1" pad="P$8"/>
-<wire x1="8.925" y1="6.215" x2="10.115" y2="6.215" width="0.1524" layer="1"/>
-<wire x1="10.115" y1="6.215" x2="10.22" y2="6.11" width="0.1524" layer="1"/>
-<wire x1="7.625" y1="6.215" x2="7.625" y2="6.2882875" width="0.1524" layer="1"/>
-<wire x1="7.625" y1="6.2882875" x2="7.8279125" y2="6.669" width="0.1524" layer="1"/>
-<wire x1="8.723678125" y1="6.669" x2="7.8279125" y2="6.669" width="0.1524" layer="1"/>
-<wire x1="8.925" y1="6.215" x2="8.925" y2="6.442278125" width="0.1524" layer="1"/>
-<wire x1="8.925" y1="6.442278125" x2="8.723678125" y2="6.669" width="0.1524" layer="1"/>
+<wire x1="2.525" y1="2.325" x2="2.525" y2="2.925" width="0.1524" layer="1"/>
+<wire x1="2.525" y1="2.925" x2="2.55" y2="2.95" width="0.1524" layer="1"/>
+<wire x1="2.55" y1="2.95" x2="3.8" y2="2.95" width="0.1524" layer="1"/>
+<wire x1="3.8" y1="2.95" x2="3.8" y2="2.35" width="0.1524" layer="1"/>
+<wire x1="3.8" y1="2.35" x2="3.825" y2="2.325" width="0.1524" layer="1"/>
+<wire x1="3.825" y1="2.325" x2="4.927" y2="2.325" width="0.1524" layer="1"/>
+<wire x1="4.927" y1="2.325" x2="4.966" y2="2.364" width="0.1524" layer="1"/>
 </signal>
 </signals>
