File: PressureSensors/Amphenol_NPA201/amphenol_npa201_pan.brd (EAGLE design)
At the start: 100 x 100 mm, 630 parts

Commit message: few changes
Parts:
- removed U$351, U$352, U$353, U$354, U$356, U$357, U$358, U$359, U$361, U$362, U$363, U$364, U$366, U$367, U$368, U$369, U$371, U$372, U$373, U$374, U$376, U$377, U$378, U$379, U$381, U$382, U$383, U$384, U$386, U$387, U$388, U$389, U$391, U$392, U$393, U$394, U$396, U$397, U$398, U$399, U$401, U$402, U$403, U$404, U$406, U$407, U$408, U$409, U$411, U$412, U$413, U$414, U$416, U$417, U$418, U$419, U$421, U$422, U$423, U$424, U$426, U$427, U$428, U$429, U$431, U$432, U$433, U$434, U$436, U$437, U$438, U$439, U$441, U$442, U$443, U$444, U$446, U$447, U$448, U$449, U$451, U$452, U$453, U$454, U$456, U$457, U$458, U$459, U$461, U$462, U$463, U$464, U$466, U$467, U$468, U$469, U$471, U$472, U$473, U$474, U$476, U$477, U$478, U$479, U$481, U$482, U$483, U$484, U$486, U$487, U$488, U$489, U$491, U$492, U$493, U$494, U$496, U$497, U$498, U$499, U$501, U$502, U$503, U$504, U$506, U$507, U$508, U$509, U$511, U$512, U$513, U$514, U$516, U$517, U$518, U$519, U$521, U$522, U$523, U$524, U$526, U$527, U$528, U$529, U$531, U$532, U$533, U$534, U$536, U$537, U$538, U$539, U$541, U$542, U$543, U$544, U$546, U$547, U$548, U$549, U$551, U$552, U$553, U$554, U$556, U$557, U$558, U$559, U$561, U$562, U$563, U$564, U$566, U$567, U$568, U$569, U$571, U$572, U$573, U$574, U$576, U$577, U$578, U$579, U$581, U$582, U$583, U$584, U$586, U$587, U$588, U$589, U$591, U$592, U$593, U$594, U$596, U$597, U$598, U$599, U$601, U$602, U$603, U$604, U$606, U$607, U$608, U$609, U$611, U$612, U$613, U$614, U$616, U$617, U$618, U$619, U$621, U$622, U$623, U$624, U$626, U$627, U$628, U$629: WIREPAD_0,8/0,45, wirepad_08-045:WIREPAD_0,8/0,45
- removed U$355, U$360, U$365, U$370, U$375, U$380, U$385, U$390, U$395, U$400, U$405, U$410, U$415, U$420, U$425, U$430, U$435, U$440, U$445, U$450, U$455, U$460, U$465, U$470, U$475, U$480, U$485, U$490, U$495, U$500, U$505, U$510, U$515, U$520, U$525, U$530, U$535, U$540, U$545, U$550, U$555, U$560, U$565, U$570, U$575, U$580, U$585, U$590, U$595, U$600, U$605, U$610, U$615, U$620, U$625, U$630: AMPHENOL_NPA201, Amphenol_NPA201:AMPHENOL_NPA201
- moved U$202 88.6 mm to (63.8, 7.86)
- moved U$204 88.5 mm to (68.0, 7.86)
- moved U$205 88.5 mm to (65.8, 8.60)
- moved U$201 88.4 mm to (63.8, 9.36)
- moved U$203 88.3 mm to (68.0, 9.36)
- moved U$207 85.9 mm to (63.8, 16.9)
- moved U$209 85.8 mm to (68.0, 16.9)
- moved U$210 85.8 mm to (65.8, 17.6)
- moved U$206 85.7 mm to (63.8, 18.4)
- moved U$208 85.6 mm to (68.0, 18.4)
- moved U$146 78.8 mm to (36.8, 91.4)
- moved U$148 78.7 mm to (41.0, 91.4)
- moved U$150 78.6 mm to (38.9, 90.6)
- moved U$147 78.5 mm to (36.8, 89.9)
- moved U$149 78.5 mm to (41.0, 89.9)
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Connections:
- removed net +3V100: U$498.P$1, U$500.P$6, U$500.P$8
- removed net +3V101: U$503.P$1, U$505.P$6, U$505.P$8
- removed net +3V102: U$508.P$1, U$510.P$6, U$510.P$8
- removed net +3V103: U$513.P$1, U$515.P$6, U$515.P$8
- removed net +3V104: U$518.P$1, U$520.P$6, U$520.P$8
- removed net +3V105: U$523.P$1, U$525.P$6, U$525.P$8
- removed net +3V106: U$528.P$1, U$530.P$6, U$530.P$8
- removed net +3V107: U$533.P$1, U$535.P$6, U$535.P$8
- removed net +3V108: U$538.P$1, U$540.P$6, U$540.P$8
- removed net +3V109: U$543.P$1, U$545.P$6, U$545.P$8
- removed net +3V110: U$548.P$1, U$550.P$6, U$550.P$8
- removed net +3V111: U$553.P$1, U$555.P$6, U$555.P$8
- removed net +3V112: U$558.P$1, U$560.P$6, U$560.P$8
- removed net +3V113: U$563.P$1, U$565.P$6, U$565.P$8
- removed net +3V114: U$568.P$1, U$570.P$6, U$570.P$8
- removed net +3V115: U$573.P$1, U$575.P$6, U$575.P$8
- removed net +3V116: U$578.P$1, U$580.P$6, U$580.P$8
- removed net +3V117: U$583.P$1, U$585.P$6, U$585.P$8
- removed net +3V118: U$588.P$1, U$590.P$6, U$590.P$8
- removed net +3V119: U$593.P$1, U$595.P$6, U$595.P$8
- removed net +3V120: U$598.P$1, U$600.P$6, U$600.P$8
- removed net +3V121: U$603.P$1, U$605.P$6, U$605.P$8
- removed net +3V122: U$608.P$1, U$610.P$6, U$610.P$8
- removed net +3V123: U$613.P$1, U$615.P$6, U$615.P$8
- removed net +3V124: U$618.P$1, U$620.P$6, U$620.P$8
- removed net +3V125: U$623.P$1, U$625.P$6, U$625.P$8
- removed net +3V126: U$628.P$1, U$630.P$6, U$630.P$8
- removed net +3V71: U$353.P$1, U$355.P$6, U$355.P$8
- removed net +3V72: U$358.P$1, U$360.P$6, U$360.P$8
- removed net +3V73: U$363.P$1, U$365.P$6, U$365.P$8
- removed net +3V74: U$368.P$1, U$370.P$6, U$370.P$8
- removed net +3V75: U$373.P$1, U$375.P$6, U$375.P$8
- removed net +3V76: U$378.P$1, U$380.P$6, U$380.P$8
- removed net +3V77: U$383.P$1, U$385.P$6, U$385.P$8
- removed net +3V78: U$388.P$1, U$390.P$6, U$390.P$8
- removed net +3V79: U$393.P$1, U$395.P$6, U$395.P$8
- removed net +3V80: U$398.P$1, U$400.P$6, U$400.P$8
- removed net +3V81: U$403.P$1, U$405.P$6, U$405.P$8
- removed net +3V82: U$408.P$1, U$410.P$6, U$410.P$8
- removed net +3V83: U$413.P$1, U$415.P$6, U$415.P$8
- removed net +3V84: U$418.P$1, U$420.P$6, U$420.P$8
- removed net +3V85: U$423.P$1, U$425.P$6, U$425.P$8
- removed net +3V86: U$428.P$1, U$430.P$6, U$430.P$8
- removed net +3V87: U$433.P$1, U$435.P$6, U$435.P$8
- removed net +3V88: U$438.P$1, U$440.P$6, U$440.P$8
- removed net +3V89: U$443.P$1, U$445.P$6, U$445.P$8
- removed net +3V90: U$448.P$1, U$450.P$6, U$450.P$8
- removed net +3V91: U$453.P$1, U$455.P$6, U$455.P$8
- removed net +3V92: U$458.P$1, U$460.P$6, U$460.P$8
- removed net +3V93: U$463.P$1, U$465.P$6, U$465.P$8
- removed net +3V94: U$468.P$1, U$470.P$6, U$470.P$8
- removed net +3V95: U$473.P$1, U$475.P$6, U$475.P$8
- removed net +3V96: U$478.P$1, U$480.P$6, U$480.P$8
- removed net +3V97: U$483.P$1, U$485.P$6, U$485.P$8
- removed net +3V98: U$488.P$1, U$490.P$6, U$490.P$8
- removed net +3V99: U$493.P$1, U$495.P$6, U$495.P$8
- removed net GND100: U$504.P$1, U$505.P$1, U$505.P$7
- removed net GND101: U$509.P$1, U$510.P$1, U$510.P$7
- removed net GND102: U$514.P$1, U$515.P$1, U$515.P$7
- removed net GND103: U$519.P$1, U$520.P$1, U$520.P$7
- removed net GND104: U$524.P$1, U$525.P$1, U$525.P$7
- removed net GND105: U$529.P$1, U$530.P$1, U$530.P$7
- removed net GND106: U$534.P$1, U$535.P$1, U$535.P$7
- removed net GND107: U$539.P$1, U$540.P$1, U$540.P$7
- removed net GND108: U$544.P$1, U$545.P$1, U$545.P$7
- removed net GND109: U$549.P$1, U$550.P$1, U$550.P$7
- removed net GND110: U$554.P$1, U$555.P$1, U$555.P$7
- removed net GND111: U$559.P$1, U$560.P$1, U$560.P$7
- removed net GND112: U$564.P$1, U$565.P$1, U$565.P$7
- removed net GND113: U$569.P$1, U$570.P$1, U$570.P$7
- removed net GND114: U$574.P$1, U$575.P$1, U$575.P$7
- removed net GND115: U$579.P$1, U$580.P$1, U$580.P$7
- removed net GND116: U$584.P$1, U$585.P$1, U$585.P$7
- removed net GND117: U$589.P$1, U$590.P$1, U$590.P$7
- removed net GND118: U$594.P$1, U$595.P$1, U$595.P$7
- removed net GND119: U$599.P$1, U$600.P$1, U$600.P$7
- removed net GND120: U$604.P$1, U$605.P$1, U$605.P$7
- removed net GND121: U$609.P$1, U$610.P$1, U$610.P$7
- removed net GND122: U$614.P$1, U$615.P$1, U$615.P$7
- removed net GND123: U$619.P$1, U$620.P$1, U$620.P$7
- removed net GND124: U$624.P$1, U$625.P$1, U$625.P$7
- removed net GND125: U$629.P$1, U$630.P$1, U$630.P$7
- removed net GND70: U$354.P$1, U$355.P$1, U$355.P$7
- removed net GND71: U$359.P$1, U$360.P$1, U$360.P$7
- removed net GND72: U$364.P$1, U$365.P$1, U$365.P$7
- removed net GND73: U$369.P$1, U$370.P$1, U$370.P$7
- removed net GND74: U$374.P$1, U$375.P$1, U$375.P$7
- removed net GND75: U$379.P$1, U$380.P$1, U$380.P$7
- removed net GND76: U$384.P$1, U$385.P$1, U$385.P$7
- removed net GND77: U$389.P$1, U$390.P$1, U$390.P$7
- removed net GND78: U$394.P$1, U$395.P$1, U$395.P$7
- removed net GND79: U$399.P$1, U$400.P$1, U$400.P$7
- removed net GND80: U$404.P$1, U$405.P$1, U$405.P$7
- removed net GND81: U$409.P$1, U$410.P$1, U$410.P$7
- removed net GND82: U$414.P$1, U$415.P$1, U$415.P$7
- removed net GND83: U$419.P$1, U$420.P$1, U$420.P$7
- removed net GND84: U$424.P$1, U$425.P$1, U$425.P$7
- removed net GND85: U$429.P$1, U$430.P$1, U$430.P$7
- removed net GND86: U$434.P$1, U$435.P$1, U$435.P$7
- removed net GND87: U$439.P$1, U$440.P$1, U$440.P$7
- removed net GND88: U$444.P$1, U$445.P$1, U$445.P$7
- removed net GND89: U$449.P$1, U$450.P$1, U$450.P$7
- removed net GND90: U$454.P$1, U$455.P$1, U$455.P$7
- removed net GND91: U$459.P$1, U$460.P$1, U$460.P$7
- removed net GND92: U$464.P$1, U$465.P$1, U$465.P$7
- removed net GND93: U$469.P$1, U$470.P$1, U$470.P$7
- removed net GND94: U$474.P$1, U$475.P$1, U$475.P$7
- removed net GND95: U$479.P$1, U$480.P$1, U$480.P$7
- removed net GND96: U$484.P$1, U$485.P$1, U$485.P$7
- removed net GND97: U$489.P$1, U$490.P$1, U$490.P$7
- removed net GND98: U$494.P$1, U$495.P$1, U$495.P$7
- removed net GND99: U$499.P$1, U$500.P$1, U$500.P$7
- removed net N$141: U$351.P$1, U$355.P$3
- removed net N$142: U$352.P$1, U$355.P$4
- removed net N$143: U$356.P$1, U$360.P$3
- removed net N$144: U$357.P$1, U$360.P$4
- removed net N$145: U$361.P$1, U$365.P$3
- removed net N$146: U$362.P$1, U$365.P$4
- removed net N$147: U$366.P$1, U$370.P$3
- removed net N$148: U$367.P$1, U$370.P$4
- removed net N$149: U$371.P$1, U$375.P$3
- removed net N$150: U$372.P$1, U$375.P$4
- removed net N$151: U$376.P$1, U$380.P$3
- removed net N$152: U$377.P$1, U$380.P$4
- removed net N$153: U$381.P$1, U$385.P$3
- removed net N$154: U$382.P$1, U$385.P$4
- removed net N$155: U$386.P$1, U$390.P$3
- removed net N$156: U$387.P$1, U$390.P$4
- removed net N$157: U$391.P$1, U$395.P$3
- removed net N$158: U$392.P$1, U$395.P$4
- removed net N$159: U$396.P$1, U$400.P$3
- removed net N$160: U$397.P$1, U$400.P$4
- removed net N$161: U$401.P$1, U$405.P$3
- removed net N$162: U$402.P$1, U$405.P$4
- removed net N$163: U$406.P$1, U$410.P$3
- removed net N$164: U$407.P$1, U$410.P$4
- removed net N$165: U$411.P$1, U$415.P$3
- removed net N$166: U$412.P$1, U$415.P$4
- removed net N$167: U$416.P$1, U$420.P$3
- removed net N$168: U$417.P$1, U$420.P$4
- removed net N$169: U$421.P$1, U$425.P$3
- removed net N$170: U$422.P$1, U$425.P$4
- removed net N$171: U$426.P$1, U$430.P$3
- removed net N$172: U$427.P$1, U$430.P$4
- removed net N$173: U$431.P$1, U$435.P$3
- removed net N$174: U$432.P$1, U$435.P$4
- removed net N$175: U$436.P$1, U$440.P$3
- removed net N$176: U$437.P$1, U$440.P$4
- removed net N$177: U$441.P$1, U$445.P$3
- removed net N$178: U$442.P$1, U$445.P$4
- removed net N$179: U$446.P$1, U$450.P$3
- removed net N$180: U$447.P$1, U$450.P$4
- removed net N$181: U$451.P$1, U$455.P$3
- removed net N$182: U$452.P$1, U$455.P$4
- removed net N$183: U$456.P$1, U$460.P$3
- removed net N$184: U$457.P$1, U$460.P$4
- removed net N$185: U$461.P$1, U$465.P$3
- removed net N$186: U$462.P$1, U$465.P$4
- removed net N$187: U$466.P$1, U$470.P$3
- removed net N$188: U$467.P$1, U$470.P$4
- removed net N$189: U$471.P$1, U$475.P$3
- removed net N$190: U$472.P$1, U$475.P$4
- removed net N$191: U$476.P$1, U$480.P$3
- removed net N$192: U$477.P$1, U$480.P$4
- removed net N$193: U$481.P$1, U$485.P$3
- removed net N$194: U$482.P$1, U$485.P$4
- removed net N$195: U$486.P$1, U$490.P$3
- removed net N$196: U$487.P$1, U$490.P$4
- removed net N$197: U$491.P$1, U$495.P$3
- removed net N$198: U$492.P$1, U$495.P$4
- removed net N$199: U$496.P$1, U$500.P$3
- removed net N$200: U$497.P$1, U$500.P$4
- removed net N$201: U$501.P$1, U$505.P$3
- removed net N$202: U$502.P$1, U$505.P$4
- removed net N$203: U$506.P$1, U$510.P$3
- removed net N$204: U$507.P$1, U$510.P$4
- removed net N$205: U$511.P$1, U$515.P$3
- removed net N$206: U$512.P$1, U$515.P$4
- removed net N$207: U$516.P$1, U$520.P$3
- removed net N$208: U$517.P$1, U$520.P$4
- removed net N$209: U$521.P$1, U$525.P$3
- removed net N$210: U$522.P$1, U$525.P$4
- removed net N$211: U$526.P$1, U$530.P$3
- removed net N$212: U$527.P$1, U$530.P$4
- removed net N$213: U$531.P$1, U$535.P$3
- removed net N$214: U$532.P$1, U$535.P$4
- removed net N$215: U$536.P$1, U$540.P$3
- removed net N$216: U$537.P$1, U$540.P$4
- removed net N$217: U$541.P$1, U$545.P$3
- removed net N$218: U$542.P$1, U$545.P$4
- removed net N$219: U$546.P$1, U$550.P$3
- removed net N$220: U$547.P$1, U$550.P$4
- removed net N$221: U$551.P$1, U$555.P$3
- removed net N$222: U$552.P$1, U$555.P$4
- removed net N$223: U$556.P$1, U$560.P$3
- removed net N$224: U$557.P$1, U$560.P$4
- removed net N$225: U$561.P$1, U$565.P$3
- removed net N$226: U$562.P$1, U$565.P$4
- removed net N$227: U$566.P$1, U$570.P$3
- removed net N$228: U$567.P$1, U$570.P$4
- removed net N$229: U$571.P$1, U$575.P$3
- removed net N$230: U$572.P$1, U$575.P$4
- removed net N$231: U$576.P$1, U$580.P$3
- removed net N$232: U$577.P$1, U$580.P$4
- removed net N$233: U$581.P$1, U$585.P$3
- removed net N$234: U$582.P$1, U$585.P$4
- removed net N$235: U$586.P$1, U$590.P$3
- removed net N$236: U$587.P$1, U$590.P$4
- removed net N$237: U$591.P$1, U$595.P$3
- removed net N$238: U$592.P$1, U$595.P$4
- removed net N$239: U$596.P$1, U$600.P$3
- removed net N$240: U$597.P$1, U$600.P$4
- removed net N$241: U$601.P$1, U$605.P$3
- removed net N$242: U$602.P$1, U$605.P$4
- removed net N$243: U$606.P$1, U$610.P$3
- removed net N$244: U$607.P$1, U$610.P$4
- removed net N$245: U$611.P$1, U$615.P$3
- removed net N$246: U$612.P$1, U$615.P$4
- removed net N$247: U$616.P$1, U$620.P$3
- removed net N$248: U$617.P$1, U$620.P$4
- removed net N$249: U$621.P$1, U$625.P$3
- removed net N$250: U$622.P$1, U$625.P$4
- removed net N$251: U$626.P$1, U$630.P$3
- removed net N$252: U$627.P$1, U$630.P$4
Routing:
- net +3V88: track 3.38 -> 0.00 mm
- net +3V87: track 3.38 -> 0.00 mm
- net +3V74: track 3.38 -> 0.00 mm
- net +3V73: track 3.38 -> 0.00 mm
- net +3V115: track 3.38 -> 0.00 mm
- net +3V114: track 3.38 -> 0.00 mm
- net +3V102: track 3.38 -> 0.00 mm
- net +3V101: track 3.38 -> 0.00 mm
- net +3V98: track 3.38 -> 0.00 mm
- net +3V97: track 3.38 -> 0.00 mm
- net +3V96: track 3.38 -> 0.00 mm
- net +3V95: track 3.38 -> 0.00 mm
- net +3V94: track 3.38 -> 0.00 mm
- net +3V86: track 3.38 -> 0.00 mm
- net +3V84: track 3.38 -> 0.00 mm
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