File: OmneticsBreakout/omnetics_nano_breakout_throughHole_v1.sch (EAGLE design)
At the start: 0 parts

Commit message: added useful helper functions for train data code
Parts:
- added U$1: FSTH-118-01-F-D, Sombeck_lib:FSTH-118-01-F-D
- added U$2: OMNETICS_NANO_18X2, Sombeck_lib:OMNETICS_NANO_18X2
Connections:
- new net AGND: U$1.P$17, U$2.REF33
- new net GND: U$1.P$18, U$1.P$20, U$2.GND0, U$2.GND34
- new net N$1: U$1.P$1, U$2.P$1
- new net N$10: U$1.P$28, U$2.P$18
- new net N$11: U$1.P$27, U$2.P$20
- new net N$12: U$1.P$26, U$2.P$22
- new net N$13: U$1.P$25, U$2.P$24
- new net N$14: U$1.P$24, U$2.P$26
- new net N$15: U$1.P$23, U$2.P$28
- new net N$16: U$1.P$22, U$2.P$30
- new net N$17: U$1.P$21, U$2.P$32
- new net N$18: U$1.P$2, U$2.P$3
- new net N$19: U$1.P$3, U$2.P$5
- new net N$2: U$1.P$36, U$2.P$2
- new net N$20: U$1.P$4, U$2.P$7
- new net N$21: U$1.P$5, U$2.P$9
- new net N$22: U$1.P$6, U$2.P$11
- new net N$23: U$1.P$7, U$2.P$13
- new net N$24: U$1.P$8, U$2.P$15
- new net N$25: U$1.P$9, U$2.P$17
- new net N$26: U$1.P$10, U$2.P$19
- new net N$27: U$1.P$11, U$2.P$21
- new net N$28: U$1.P$12, U$2.P$23
- new net N$29: U$1.P$13, U$2.P$25
- new net N$3: U$1.P$35, U$2.P$4
- new net N$30: U$1.P$14, U$2.P$27
- new net N$31: U$1.P$15, U$2.P$29
- new net N$32: U$1.P$16, U$2.P$31
- new net N$4: U$1.P$34, U$2.P$6
- new net N$5: U$1.P$33, U$2.P$8
- new net N$6: U$1.P$32, U$2.P$10
- new net N$7: U$1.P$31, U$2.P$12
- new net N$8: U$1.P$30, U$2.P$14
- new net N$9: U$1.P$29, U$2.P$16
