File: OmneticsBreakout/omnetics_nano_breakout_reverse_v2.sch (EAGLE design)
At the start: 2 parts

Commit message: omentics breakout board
Parts:
- U$1: value FTSH-118-01-L-MTINVERTED -> SFMC-118-L1-S-D; device tuckerLib:FTSH-118-01-L-MTINVERTED -> tuckerLib:SFMC-118-L1-S-D
Connections:
- new net N$19: U$1.5, U$2.P$5
- new net N$20: U$1.7, U$2.P$7
- new net N$21: U$1.9, U$2.P$9
- new net N$22: U$1.11, U$2.P$11
- new net N$23: U$1.13, U$2.P$13
- new net N$24: U$1.15, U$2.P$15
- new net N$25: U$1.17, U$2.P$17
- new net N$26: U$1.19, U$2.P$19
- new net N$27: U$1.21, U$2.P$21
- new net N$28: U$1.23, U$2.P$23
- new net N$29: U$1.25, U$2.P$25
- new net N$30: U$1.27, U$2.P$27
- new net N$31: U$1.29, U$2.P$29
- new net N$32: U$1.31, U$2.P$31
